Commit message: Add Nav2 navigation and unified simulation bringup

File: ros2_ws/src/omni_robot_description/urdf/omni_robot.urdf.xacro (robot description, xacro)
@@ -2,8 +2,10 @@
 <robot name="omni_robot" xmlns:xacro="http://www.ros.org/wiki/xacro">
   <xacro:arg name="controllers_file" default=""/>
+  <!-- Base parameters -->
   <xacro:property name="base_length" value="0.6"/>
   <xacro:property name="base_width" value="0.6"/>
   <xacro:property name="base_height" value="0.15"/>
   <xacro:property name="base_mass" value="20.0"/>
+  <!-- Wheel parameters -->
   <xacro:property name="wheel_radius" value="0.05"/>
   <xacro:property name="wheel_width" value="0.03"/>
@@ -15,5 +17,5 @@
     <parent link="base_footprint"/>
     <child link="base_link"/>
-    <origin xyz="0 0 0.075"/>
+    <origin xyz="0 0 0.075" rpy="0 0 0"/>
   </joint>
   <!-- base_link -->
@@ -28,25 +30,28 @@
     </visual>
     <collision>
-        <geometry>
-    	<box size="${base_length} ${base_width} ${base_height}"/>
-  	</geometry>
+      <geometry>
+        <box size="${base_length} ${base_width} ${base_height}"/>
+      </geometry>
     </collision>
     <inertial>
       <mass value="${base_mass}"/>
-      <origin xyz="0 0 0"/>
+      <origin xyz="0 0 0" rpy="0 0 0"/>
       <inertia
-        ixx="0.8"
+        ixx="0.6375"
         ixy="0.0"
         ixz="0.0"
-        iyy="0.8"
+        iyy="0.6375"
         iyz="0.0"
         izz="1.2"/>
     </inertial>
   </link>
+  <gazebo reference="base_link">
+    <material>Gazebo/Blue</material>
+  </gazebo>
   <!-- Wheel macro -->
   <xacro:macro name="wheel" params="name x y yaw">
     <link name="${name}">
       <visual>
-        <origin rpy="1.570796 0 0"/>
+        <origin xyz="0 0 0" rpy="1.57079632679 0 0"/>
         <geometry>
           <cylinder
@@ -59,5 +64,5 @@
       </visual>
       <collision>
-        <origin rpy="1.570796 0 0"/>
+        <origin xyz="0 0 0" rpy="1.57079632679 0 0"/>
         <geometry>
           <cylinder
@@ -68,12 +73,12 @@
       <inertial>
         <mass value="${wheel_mass}"/>
-        <origin xyz="0 0 0"/>
+        <origin xyz="0 0 0" rpy="0 0 0"/>
         <inertia
-          ixx="0.000154"
+          ixx="0.00035"
           ixy="0.0"
           ixz="0.0"
           iyy="0.000625"
           iyz="0.0"
-          izz="0.000154"/>
+          izz="0.00035"/>
       </inertial>
     </link>
@@ -85,4 +90,7 @@
         rpy="0 0 ${yaw}"/>
       <axis xyz="0 1 0"/>
+      <limit
+        effort="100.0"
+        velocity="60.0"/>
       <dynamics
         damping="0.02"
@@ -90,6 +98,8 @@
     </joint>
     <gazebo reference="${name}">
+      <material>Gazebo/Black</material>
       <mu1>1.0</mu1>
       <mu2>0.02</mu2>
+      <fdir1>1 0 0</fdir1>
       <kp>1000000.0</kp>
       <kd>10.0</kd>
@@ -103,21 +113,21 @@
     x="0.25"
     y="0.25"
-    yaw="-0.785398"/>
+    yaw="-0.78539816339"/>
   <xacro:wheel
     name="front_right_wheel"
     x="0.25"
     y="-0.25"
-    yaw="0.785398"/>
+    yaw="0.78539816339"/>
   <xacro:wheel
     name="rear_left_wheel"
     x="-0.25"
     y="0.25"
-    yaw="0.785398"/>
+    yaw="0.78539816339"/>
   <xacro:wheel
     name="rear_right_wheel"
     x="-0.25"
     y="-0.25"
-    yaw="-0.785398"/>
-  <!-- 2D LiDAR -->
+    yaw="-0.78539816339"/>
+  <!-- Visible LiDAR body -->
   <link name="lidar_link">
     <visual>
@@ -129,27 +139,23 @@
       </material>
     </visual>
-    <collision>
-      <geometry>
-        <cylinder radius="0.04" length="0.05"/>
-      </geometry>
-    </collision>
-    <inertial>
-      <mass value="0.2"/>
-      <origin xyz="0 0 0"/>
-      <inertia
-        ixx="0.0001"
-        ixy="0.0"
-        ixz="0.0"
-        iyy="0.0001"
-        iyz="0.0"
-        izz="0.0001"/>
-    </inertial>
   </link>
   <joint name="lidar_joint" type="fixed">
     <parent link="base_link"/>
     <child link="lidar_link"/>
-    <origin xyz="0.38 0 -0.10" rpy="0 0 0"/>
-  </joint>
-  <gazebo reference="lidar_link">
+    <origin xyz="0.0 0.0 0.10" rpy="0 0 0"/>
+  </joint>
+  <!--
+    Invisible scan origin.
+    The visible LiDAR remains on the robot.
+    The scan origin is placed forward and lower so that the low field walls
+    can be detected without the laser intersecting the robot body.
+  -->
+  <link name="lidar_scan_link"/>
+  <joint name="lidar_scan_joint" type="fixed">
+    <parent link="base_link"/>
+    <child link="lidar_scan_link"/>
+    <origin xyz="0.38 0.0 -0.10" rpy="0 0 0"/>
+  </joint>
+  <gazebo reference="lidar_scan_link">
     <sensor name="lidar_sensor" type="ray">
       <always_on>true</always_on>
@@ -161,6 +167,6 @@
             <samples>720</samples>
             <resolution>1.0</resolution>
-            <min_angle>-3.14159265</min_angle>
-            <max_angle>3.14159265</max_angle>
+            <min_angle>-3.14159265359</min_angle>
+            <max_angle>3.14159265359</max_angle>
           </horizontal>
         </scan>
@@ -183,5 +189,5 @@
         </ros>
         <output_type>sensor_msgs/LaserScan</output_type>
-        <frame_name>lidar_link</frame_name>
+        <frame_name>lidar_scan_link</frame_name>
       </plugin>
     </sensor>
@@ -192,5 +198,5 @@
     <parent link="base_link"/>
     <child link="imu_link"/>
-    <origin xyz="0 0 0"/>
+    <origin xyz="0 0 0" rpy="0 0 0"/>
   </joint>
   <!-- ros2_control -->

Commit message: 500mm機体で回収・配置地点までの自律移動を実装

File: ros2_ws/src/omni_robot_description/urdf/omni_robot.urdf.xacro (robot description, xacro)
@@ -3,6 +3,6 @@
   <xacro:arg name="controllers_file" default=""/>
   <!-- Base parameters -->
-  <xacro:property name="base_length" value="0.6"/>
-  <xacro:property name="base_width" value="0.6"/>
+  <xacro:property name="base_length" value="0.5"/>
+  <xacro:property name="base_width" value="0.5"/>
   <xacro:property name="base_height" value="0.15"/>
   <xacro:property name="base_mass" value="20.0"/>
@@ -111,21 +111,21 @@
   <xacro:wheel
     name="front_left_wheel"
-    x="0.25"
-    y="0.25"
+    x="0.20"
+    y="0.20"
     yaw="-0.78539816339"/>
   <xacro:wheel
     name="front_right_wheel"
-    x="0.25"
-    y="-0.25"
+    x="0.20"
+    y="-0.20"
     yaw="0.78539816339"/>
   <xacro:wheel
     name="rear_left_wheel"
-    x="-0.25"
-    y="0.25"
+    x="-0.20"
+    y="0.20"
     yaw="0.78539816339"/>
   <xacro:wheel
     name="rear_right_wheel"
-    x="-0.25"
-    y="-0.25"
+    x="-0.20"
+    y="-0.20"
     yaw="-0.78539816339"/>
   <!-- Visible LiDAR body -->
