Commit message: フェーズ1: ロボット寸法をrobot_geometry.yamlに集約し実機寸法に合わせる
- omni_robot_description/config/robot_geometry.yaml を唯一の寸法定義にし、
  URDF(xacro.load_yaml)・omni_drive_controller・omni_odometry・Nav2フットプリントがここから値を取る
- X配置4輪オムニ: L=0.2245 m、車輪直径0.125 m、幅0.04 m、総質量20 kg、台車0.5 m角
- 最大外形(max_outline)を台車外形と別パラメータにし、フットプリントはそちらを使う(仮値0.5 m)
- base_footprintを床面に合わせ、慣性を直方体・円柱から計算
- 車輪速度をvelocity_pid(トルク上限つき)で駆動。従来のSetVelocity方式では負荷で車輪速度が
  指令の約6割に落ち、並進がほとんど追従しなかった
- オムニ輪の摩擦方向fdir1を車軸方向(回転しても向きが変わらない)で指定
- 真値取得用にp3dプラグイン(/ground_truth/odom)を追加
- wheel_geometry.yamlは削除し、Gazeboのスポーン姿勢とGUI有無を起動引数にした

Co-Authored-By: Claude Opus 5.5 <noreply@anthropic.com>

File: ros2_ws/src/omni_robot_description/urdf/omni_robot.urdf.xacro (robot description, xacro)
@@ -1,23 +1,33 @@
 <?xml version="1.0"?>
 <robot name="omni_robot" xmlns:xacro="http://www.ros.org/wiki/xacro">
+  <!-- Comments must not contain colon-space. gazebo_ros2_control parses the
+       whole description as a YAML parameter value. -->
   <xacro:arg name="controllers_file" default=""/>
-  <!-- Base parameters -->
-  <xacro:property name="base_length" value="0.5"/>
-  <xacro:property name="base_width" value="0.5"/>
-  <xacro:property name="base_height" value="0.15"/>
-  <xacro:property name="base_mass" value="20.0"/>
-  <!-- Wheel parameters -->
-  <xacro:property name="wheel_radius" value="0.05"/>
-  <xacro:property name="wheel_width" value="0.03"/>
-  <xacro:property name="wheel_mass" value="0.5"/>
-  <xacro:property name="wheel_z" value="-0.075"/>
-  <!-- base_footprint -->
+  <xacro:arg name="geometry_file"
+    default="$(find omni_robot_description)/config/robot_geometry.yaml"/>
+  <!-- All dimensions come from robot_geometry.yaml -->
+  <xacro:property name="geom" value="${xacro.load_yaml('$(arg geometry_file)')}"/>
+  <xacro:property name="base_length" value="${geom['chassis']['length']}"/>
+  <xacro:property name="base_width" value="${geom['chassis']['width']}"/>
+  <xacro:property name="base_height" value="${geom['chassis']['height']}"/>
+  <xacro:property name="base_center_z"
+    value="${geom['chassis']['ground_clearance'] + 0.5 * base_height}"/>
+  <xacro:property name="wheel_radius" value="${0.5 * geom['drive_wheels']['diameter']}"/>
+  <xacro:property name="wheel_width" value="${geom['drive_wheels']['width']}"/>
+  <xacro:property name="wheel_mass" value="${geom['mass']['drive_wheel']}"/>
+  <xacro:property name="wheel_distance" value="${geom['drive_wheels']['center_distance']}"/>
+  <!-- Wheel axle height relative to base_link (base_footprint is on the floor) -->
+  <xacro:property name="wheel_z" value="${wheel_radius - base_center_z}"/>
+  <xacro:property name="max_wheel_speed" value="${geom['drive_wheels']['max_wheel_speed']}"/>
+  <!-- Chassis carries the remaining mass -->
+  <xacro:property name="base_mass" value="${geom['mass']['total'] - 4 * wheel_mass}"/>
+  <!-- base_footprint on the floor, below the robot center -->
   <link name="base_footprint"/>
   <joint name="base_footprint_joint" type="fixed">
     <parent link="base_footprint"/>
     <child link="base_link"/>
-    <origin xyz="0 0 0.075" rpy="0 0 0"/>
+    <origin xyz="0 0 ${base_center_z}" rpy="0 0 0"/>
   </joint>
-  <!-- base_link -->
+  <!-- base_link at the chassis center -->
   <link name="base_link">
     <visual>
@@ -37,11 +47,12 @@
       <mass value="${base_mass}"/>
       <origin xyz="0 0 0" rpy="0 0 0"/>
+      <!-- Solid box -->
       <inertia
-        ixx="0.6375"
+        ixx="${base_mass * (base_width**2 + base_height**2) / 12.0}"
         ixy="0.0"
         ixz="0.0"
-        iyy="0.6375"
+        iyy="${base_mass * (base_length**2 + base_height**2) / 12.0}"
         iyz="0.0"
-        izz="1.2"/>
+        izz="${base_mass * (base_length**2 + base_width**2) / 12.0}"/>
     </inertial>
   </link>
@@ -49,9 +60,13 @@
     <material>Gazebo/Blue</material>
   </gazebo>
-  <!-- Wheel macro -->
-  <xacro:macro name="wheel" params="name x y yaw">
+  <!-- Wheel macro. index selects the entry in robot_geometry.yaml -->
+  <xacro:macro name="wheel" params="index">
+    <xacro:property name="name"
+      value="${geom['drive_wheels']['names'][index]}_wheel"/>
+    <xacro:property name="angle"
+      value="${radians(geom['drive_wheels']['position_angles_deg'][index])}"/>
     <link name="${name}">
       <visual>
-        <origin xyz="0 0 0" rpy="1.57079632679 0 0"/>
+        <origin xyz="0 0 0" rpy="${pi / 2} 0 0"/>
         <geometry>
           <cylinder
@@ -64,5 +79,5 @@
       </visual>
       <collision>
-        <origin xyz="0 0 0" rpy="1.57079632679 0 0"/>
+        <origin xyz="0 0 0" rpy="${pi / 2} 0 0"/>
         <geometry>
           <cylinder
@@ -74,23 +89,26 @@
         <mass value="${wheel_mass}"/>
         <origin xyz="0 0 0" rpy="0 0 0"/>
+        <!-- Solid cylinder, axle along y -->
         <inertia
-          ixx="0.00035"
+          ixx="${wheel_mass * (3 * wheel_radius**2 + wheel_width**2) / 12.0}"
           ixy="0.0"
           ixz="0.0"
-          iyy="0.000625"
+          iyy="${wheel_mass * wheel_radius**2 / 2.0}"
           iyz="0.0"
-          izz="0.00035"/>
+          izz="${wheel_mass * (3 * wheel_radius**2 + wheel_width**2) / 12.0}"/>
       </inertial>
     </link>
+    <!-- Axle is radial (local y), so the rolling direction is angle - 90 deg.
+         Diagonal wheels share one axle line through the center. -->
     <joint name="${name}_joint" type="continuous">
       <parent link="base_link"/>
       <child link="${name}"/>
       <origin
-        xyz="${x} ${y} ${wheel_z}"
-        rpy="0 0 ${yaw}"/>
+        xyz="${wheel_distance * cos(angle)} ${wheel_distance * sin(angle)} ${wheel_z}"
+        rpy="0 0 ${atan2(sin(angle - pi / 2), cos(angle - pi / 2))}"/>
       <axis xyz="0 1 0"/>
       <limit
-        effort="100.0"
-        velocity="60.0"/>
+        effort="${geom['drive_wheels']['max_wheel_torque']}"
+        velocity="${max_wheel_speed * 1.5}"/>
       <dynamics
         damping="0.02"
@@ -99,7 +117,10 @@
     <gazebo reference="${name}">
       <material>Gazebo/Black</material>
-      <mu1>1.0</mu1>
-      <mu2>0.02</mu2>
-      <fdir1>1 0 0</fdir1>
+      <!-- Omni wheel approximation. fdir1 is given in the collision frame,
+           where z is the axle. The axle does not turn while the wheel spins,
+           so mu1 stays along the free rollers and mu2 along rolling. -->
+      <mu1>${geom['drive_wheels']['mu_axle']}</mu1>
+      <mu2>${geom['drive_wheels']['mu_rolling']}</mu2>
+      <fdir1>0 0 1</fdir1>
       <kp>1000000.0</kp>
       <kd>10.0</kd>
@@ -108,25 +129,9 @@
     </gazebo>
   </xacro:macro>
-  <!-- Four omni wheels -->
-  <xacro:wheel
-    name="front_left_wheel"
-    x="0.20"
-    y="0.20"
-    yaw="-0.78539816339"/>
-  <xacro:wheel
-    name="front_right_wheel"
-    x="0.20"
-    y="-0.20"
-    yaw="0.78539816339"/>
-  <xacro:wheel
-    name="rear_left_wheel"
-    x="-0.20"
-    y="0.20"
-    yaw="0.78539816339"/>
-  <xacro:wheel
-    name="rear_right_wheel"
-    x="-0.20"
-    y="-0.20"
-    yaw="-0.78539816339"/>
+  <!-- Four omni wheels in X configuration -->
+  <xacro:wheel index="0"/>
+  <xacro:wheel index="1"/>
+  <xacro:wheel index="2"/>
+  <xacro:wheel index="3"/>
   <!-- Visible LiDAR body -->
   <link name="lidar_link">
@@ -198,5 +203,5 @@
     <parent link="base_link"/>
     <child link="imu_link"/>
-    <origin xyz="0 0 0" rpy="0 0 0"/>
+    <origin xyz="${geom['imu']['xyz'][0]} ${geom['imu']['xyz'][1]} ${geom['imu']['xyz'][2]}" rpy="0 0 0"/>
   </joint>
   <gazebo reference="imu_link">
@@ -258,41 +263,43 @@
     </sensor>
   </gazebo>
+  <!-- Ground truth pose of base_footprint (simulation only) -->
+  <gazebo>
+    <plugin name="ground_truth_p3d" filename="libgazebo_ros_p3d.so">
+      <ros>
+        <remapping>odom:=ground_truth/odom</remapping>
+      </ros>
+      <body_name>base_footprint</body_name>
+      <frame_name>world</frame_name>
+      <update_rate>100.0</update_rate>
+      <gaussian_noise>0.0</gaussian_noise>
+    </plugin>
+  </gazebo>
   <!-- ros2_control -->
+  <xacro:macro name="velocity_joint" params="index">
+    <xacro:property name="pid" value="${geom['drive_wheels']['velocity_pid']}"/>
+    <joint name="${geom['drive_wheels']['names'][index]}_wheel_joint">
+      <!-- velocity_pid turns the velocity command into joint torque limited
+           by the joint effort limit, like a motor with a speed controller -->
+      <param name="vel_kp">${pid['kp']}</param>
+      <param name="vel_ki">${pid['ki']}</param>
+      <param name="vel_kd">${pid['kd']}</param>
+      <param name="vel_max_integral_error">${pid['max_integral_error']}</param>
+      <param name="vel_min_integral_error">${-pid['max_integral_error']}</param>
+      <command_interface name="velocity_pid">
+        <param name="min">${-max_wheel_speed * 1.5}</param>
+        <param name="max">${max_wheel_speed * 1.5}</param>
+      </command_interface>
+      <state_interface name="position"/>
+      <state_interface name="velocity"/>
+    </joint>
+  </xacro:macro>
   <ros2_control name="GazeboSystem" type="system">
     <hardware>
       <plugin>gazebo_ros2_control/GazeboSystem</plugin>
     </hardware>
-    <joint name="front_left_wheel_joint">
-      <command_interface name="velocity">
-        <param name="min">-60.0</param>
-        <param name="max">60.0</param>
-      </command_interface>
-      <state_interface name="position"/>
-      <state_interface name="velocity"/>
-    </joint>
-    <joint name="front_right_wheel_joint">
-      <command_interface name="velocity">
-        <param name="min">-60.0</param>
-        <param name="max">60.0</param>
-      </command_interface>
-      <state_interface name="position"/>
-      <state_interface name="velocity"/>
-    </joint>
-    <joint name="rear_left_wheel_joint">
-      <command_interface name="velocity">
-        <param name="min">-60.0</param>
-        <param name="max">60.0</param>
-      </command_interface>
-      <state_interface name="position"/>
-      <state_interface name="velocity"/>
-    </joint>
-    <joint name="rear_right_wheel_joint">
-      <command_interface name="velocity">
-        <param name="min">-60.0</param>
-        <param name="max">60.0</param>
-      </command_interface>
-      <state_interface name="position"/>
-      <state_interface name="velocity"/>
-    </joint>
+    <xacro:velocity_joint index="0"/>
+    <xacro:velocity_joint index="1"/>
+    <xacro:velocity_joint index="2"/>
+    <xacro:velocity_joint index="3"/>
   </ros2_control>
   <!-- gazebo_ros2_control -->

Commit message: フェーズ2: フィールドをルールブック寸法で作り直し、LiDARを実機想定に変更
- config/field_layout.yaml(図4の寸法、赤コート)からGazeboのSDFとNav2マップを生成する
  field_layout.py(generate_field)を追加。木枠38x89 mmのbox、床z=0、白線は見た目のみ
- 既存STLとの差: 床が80 mmの台・木枠が床上38 mm・エリア1上枠が76 mm下・白線が溝だった
- LiDARをUTM-30LX-EW相当(270度,1081点,40 Hz,0.1-30 m)に変更。取り付け面・高さ・
  逆さ取り付けはrobot_geometry.yaml、取り付け誤差はsim_conditions.yamlで与え、
  誤差はGazeboにスポーンするモデルだけに入れる(TFは設計値のまま)
- laser_filtersで自機に当たる角度(±88度より外側、仮値)をマスクし/scan_filteredを出す。
  AMCLとコストマップの入力を/scan_filteredに変更
- 確認用のsim_check.launch.py(Gazebo GUI+RViz、サイコロゾーン前にスポーン)とRViz設定、
  ルート上の壁の見え方を数えるscan_visibility_checkを追加

Co-Authored-By: Claude Opus 5.5 <noreply@anthropic.com>

File: ros2_ws/src/omni_robot_description/urdf/omni_robot.urdf.xacro (robot description, xacro)
@@ -134,55 +134,72 @@
   <xacro:wheel index="2"/>
   <xacro:wheel index="3"/>
-  <!-- Visible LiDAR body -->
-  <link name="lidar_link">
+  <!-- LiDAR (Hokuyo UTM-30LX-EW). Mounting from robot_geometry.yaml.
+       lidar_mount_link is the nominal pose (what the robot believes).
+       lidar_scan_link adds the mounting error, which is non-zero only in
+       the model spawned in Gazebo (sim_conditions.yaml). -->
+  <xacro:property name="lidar" value="${geom['lidar']}"/>
+  <xacro:property name="mount" value="${lidar['mount']}"/>
+  <xacro:property name="face_yaw"
+    value="${0.0 if mount['face'] == '+x' else (pi / 2 if mount['face'] == '+y' else (pi if mount['face'] == '-x' else -pi / 2))}"/>
+  <xacro:property name="face_half"
+    value="${0.5 * base_length if mount['face'] in ('+x', '-x') else 0.5 * base_width}"/>
+  <xacro:property name="lidar_out" value="${face_half + mount['outward_offset']}"/>
+  <xacro:property name="lidar_side" value="${mount['lateral_offset']}"/>
+  <xacro:arg name="lidar_err_x" default="0.0"/>
+  <xacro:arg name="lidar_err_y" default="0.0"/>
+  <xacro:arg name="lidar_err_z" default="0.0"/>
+  <xacro:arg name="lidar_err_roll_deg" default="0.0"/>
+  <xacro:arg name="lidar_err_pitch_deg" default="0.0"/>
+  <xacro:arg name="lidar_err_yaw_deg" default="0.0"/>
+  <link name="lidar_mount_link"/>
+  <joint name="lidar_mount_joint" type="fixed">
+    <parent link="base_link"/>
+    <child link="lidar_mount_link"/>
+    <origin
+      xyz="${lidar_out * cos(face_yaw) - lidar_side * sin(face_yaw)} ${lidar_out * sin(face_yaw) + lidar_side * cos(face_yaw)} ${mount['scan_height'] - base_center_z}"
+      rpy="${pi if mount['upside_down'] else 0.0} 0 ${face_yaw}"/>
+  </joint>
+  <link name="lidar_scan_link">
     <visual>
+      <!-- Sensor body centered on the scan plane -->
       <geometry>
-        <cylinder radius="0.04" length="0.05"/>
+        <box size="${lidar['body_size'][0]} ${lidar['body_size'][1]} ${lidar['body_size'][2]}"/>
       </geometry>
-      <material name="green">
-        <color rgba="0.0 1.0 0.0 1.0"/>
+      <material name="dark_gray">
+        <color rgba="0.2 0.2 0.2 1.0"/>
       </material>
     </visual>
   </link>
-  <joint name="lidar_joint" type="fixed">
-    <parent link="base_link"/>
-    <child link="lidar_link"/>
-    <origin xyz="0.0 0.0 0.10" rpy="0 0 0"/>
-  </joint>
-  <!--
-    Invisible scan origin.
-    The visible LiDAR remains on the robot.
-    The scan origin is placed forward and lower so that the low field walls
-    can be detected without the laser intersecting the robot body.
-  -->
-  <link name="lidar_scan_link"/>
   <joint name="lidar_scan_joint" type="fixed">
-    <parent link="base_link"/>
+    <parent link="lidar_mount_link"/>
     <child link="lidar_scan_link"/>
-    <origin xyz="0.38 0.0 -0.10" rpy="0 0 0"/>
+    <origin
+      xyz="$(arg lidar_err_x) $(arg lidar_err_y) $(arg lidar_err_z)"
+      rpy="${radians($(arg lidar_err_roll_deg))} ${radians($(arg lidar_err_pitch_deg))} ${radians($(arg lidar_err_yaw_deg))}"/>
   </joint>
   <gazebo reference="lidar_scan_link">
+    <material>Gazebo/DarkGrey</material>
     <sensor name="lidar_sensor" type="ray">
       <always_on>true</always_on>
       <visualize>true</visualize>
-      <update_rate>10.0</update_rate>
+      <update_rate>${lidar['update_rate']}</update_rate>
       <ray>
         <scan>
           <horizontal>
-            <samples>720</samples>
+            <samples>${lidar['samples']}</samples>
             <resolution>1.0</resolution>
-            <min_angle>-3.14159265359</min_angle>
-            <max_angle>3.14159265359</max_angle>
+            <min_angle>${-radians(lidar['fov_deg']) / 2}</min_angle>
+            <max_angle>${radians(lidar['fov_deg']) / 2}</max_angle>
           </horizontal>
         </scan>
         <range>
-          <min>0.08</min>
-          <max>12.0</max>
-          <resolution>0.01</resolution>
+          <min>${lidar['range_min']}</min>
+          <max>${lidar['range_max']}</max>
+          <resolution>0.001</resolution>
         </range>
         <noise>
           <type>gaussian</type>
           <mean>0.0</mean>
-          <stddev>0.005</stddev>
+          <stddev>${lidar['noise_stddev']}</stddev>
         </noise>
       </ray>

Commit message: フェーズ3: 独立した計測輪2つとtracking_odometryを追加しEKFの入力を切り替え
- 直径50 mm(仮値)の受動オムニ輪をx方向用・y方向用に直交配置。prismaticジョイント+
  バネ(2000 N/m、予圧15 N、いずれも仮値)で床に押し付ける。寸法はrobot_geometry.yaml
- 実機共通のomni_robot_odometryパッケージにtracking_odometryを追加。計測輪2つと
  IMUのヨー角速度から中心オフセットを補正して/tracking/odomを出す
  (dy = d1 - x1*dθ, dx = d2 + y2*dθ を一般の取り付け角で解く形)
- EKFのodom0を/tracking/odomに切り替え。駆動輪オドメトリ/wheel/odomは比較用に残す
- 加減速を繰り返して各オドメトリを真値と比べるodometry_comparisonを追加し、3回の結果と
  フェーズ2の壁の見え方の結果をresults/に保存

Co-Authored-By: Claude Opus 5.5 <noreply@anthropic.com>

File: ros2_ws/src/omni_robot_description/urdf/omni_robot.urdf.xacro (robot description, xacro)
@@ -20,6 +20,8 @@
   <xacro:property name="wheel_z" value="${wheel_radius - base_center_z}"/>
   <xacro:property name="max_wheel_speed" value="${geom['drive_wheels']['max_wheel_speed']}"/>
+  <xacro:property name="tracking" value="${geom['tracking_wheels']}"/>
   <!-- Chassis carries the remaining mass -->
-  <xacro:property name="base_mass" value="${geom['mass']['total'] - 4 * wheel_mass}"/>
+  <xacro:property name="base_mass"
+    value="${geom['mass']['total'] - 4 * wheel_mass - len(tracking['wheels']) * (tracking['wheel_mass'] + tracking['mount_mass'])}"/>
   <!-- base_footprint on the floor, below the robot center -->
   <link name="base_footprint"/>
@@ -134,4 +136,85 @@
   <xacro:wheel index="2"/>
   <xacro:wheel index="3"/>
+  <!-- Passive measuring (tracking) omni wheels. Each one hangs from a
+       vertical prismatic joint with a spring. At joint position 0 the wheel
+       would sink spring_preload / spring_stiffness into the floor, so on the
+       floor the spring presses it down with about spring_preload. -->
+  <xacro:property name="tw_radius" value="${0.5 * tracking['diameter']}"/>
+  <xacro:property name="tw_width" value="${tracking['width']}"/>
+  <xacro:property name="tw_preload_depth"
+    value="${tracking['spring_preload'] / tracking['spring_stiffness']}"/>
+  <xacro:macro name="tracking_wheel" params="index">
+    <xacro:property name="wheel" value="${tracking['wheels'][index]}"/>
+    <xacro:property name="name" value="${wheel['name']}"/>
+    <link name="${name}_mount">
+      <inertial>
+        <mass value="${tracking['mount_mass']}"/>
+        <inertia ixx="1e-5" ixy="0" ixz="0" iyy="1e-5" iyz="0" izz="1e-5"/>
+      </inertial>
+    </link>
+    <!-- Local x is the measuring (rolling) direction -->
+    <joint name="${name}_spring_joint" type="prismatic">
+      <parent link="base_link"/>
+      <child link="${name}_mount"/>
+      <origin
+        xyz="${wheel['xy'][0]} ${wheel['xy'][1]} ${tw_radius - tw_preload_depth - base_center_z}"
+        rpy="0 0 ${radians(wheel['rolling_deg'])}"/>
+      <axis xyz="0 0 1"/>
+      <limit lower="${-tracking['travel']}" upper="${tracking['travel']}"
+        effort="1000.0" velocity="1.0"/>
+      <dynamics damping="${tracking['spring_damping']}" friction="0.0"/>
+    </joint>
+    <gazebo reference="${name}_spring_joint">
+      <springStiffness>${tracking['spring_stiffness']}</springStiffness>
+      <springReference>0.0</springReference>
+      <implicitSpringDamper>true</implicitSpringDamper>
+    </gazebo>
+    <link name="${name}_wheel">
+      <visual>
+        <origin xyz="0 0 0" rpy="${pi / 2} 0 0"/>
+        <geometry>
+          <cylinder radius="${tw_radius}" length="${tw_width}"/>
+        </geometry>
+        <material name="orange">
+          <color rgba="1.0 0.5 0.0 1.0"/>
+        </material>
+      </visual>
+      <collision>
+        <origin xyz="0 0 0" rpy="${pi / 2} 0 0"/>
+        <geometry>
+          <cylinder radius="${tw_radius}" length="${tw_width}"/>
+        </geometry>
+      </collision>
+      <inertial>
+        <mass value="${tracking['wheel_mass']}"/>
+        <inertia
+          ixx="${tracking['wheel_mass'] * (3 * tw_radius**2 + tw_width**2) / 12.0}"
+          ixy="0" ixz="0"
+          iyy="${tracking['wheel_mass'] * tw_radius**2 / 2.0}"
+          iyz="0"
+          izz="${tracking['wheel_mass'] * (3 * tw_radius**2 + tw_width**2) / 12.0}"/>
+      </inertial>
+    </link>
+    <joint name="${name}_wheel_joint" type="continuous">
+      <parent link="${name}_mount"/>
+      <child link="${name}_wheel"/>
+      <origin xyz="0 0 0" rpy="0 0 0"/>
+      <axis xyz="0 1 0"/>
+      <dynamics damping="0.0" friction="0.0"/>
+    </joint>
+    <gazebo reference="${name}_wheel">
+      <material>Gazebo/Orange</material>
+      <!-- Same omni approximation as the drive wheels (collision z = axle) -->
+      <mu1>${tracking['mu_axle']}</mu1>
+      <mu2>${tracking['mu_rolling']}</mu2>
+      <fdir1>0 0 1</fdir1>
+      <kp>1000000.0</kp>
+      <kd>10.0</kd>
+      <minDepth>0.001</minDepth>
+      <maxVel>0.1</maxVel>
+    </gazebo>
+  </xacro:macro>
+  <xacro:tracking_wheel index="0"/>
+  <xacro:tracking_wheel index="1"/>
   <!-- LiDAR (Hokuyo UTM-30LX-EW). Mounting from robot_geometry.yaml.
        lidar_mount_link is the nominal pose (what the robot believes).
@@ -311,4 +394,13 @@
     </joint>
   </xacro:macro>
+  <xacro:macro name="tracking_joints" params="index">
+    <joint name="${tracking['wheels'][index]['name']}_wheel_joint">
+      <state_interface name="position"/>
+      <state_interface name="velocity"/>
+    </joint>
+    <joint name="${tracking['wheels'][index]['name']}_spring_joint">
+      <state_interface name="position"/>
+    </joint>
+  </xacro:macro>
   <ros2_control name="GazeboSystem" type="system">
     <hardware>
@@ -319,4 +411,7 @@
     <xacro:velocity_joint index="2"/>
     <xacro:velocity_joint index="3"/>
+    <!-- Passive tracking wheels: state only (encoders, spring travel) -->
+    <xacro:tracking_joints index="0"/>
+    <xacro:tracking_joints index="1"/>
   </ros2_control>
   <!-- gazebo_ros2_control -->
